Commit message: added joint_state_publisher to fix wheel joint transforms

File: src/robot_package/urdf/my_mobile_robot.urdf (robot description, URDF)
Before this commit: robot my_mobile_robot, 4 links, 3 joints
Links:
- link base_link: geometry visual box size=0.5 0.5 0.2
- link wheel_left: geometry visual cylinder length=0.05 radius=0.1
- link wheel_right: geometry visual cylinder length=0.05 radius=0.1
- link world: geometry visual sphere radius=0.05
Joints:
- joint left_wheel_joint: limit effort=10.0 velocity=10.0 -> lower=-1.57 upper=1.57 effort=10.0 velocity=5.0
- joint right_wheel_joint: limit effort=10.0 velocity=10.0 -> lower=-1.57 upper=1.57 effort=10.0 velocity=5.0

Commit message: Three wheeled robot from Articulated Robotics

File: src/robot_package/urdf/my_mobile_robot.urdf (robot description, URDF)
Before this commit: robot my_mobile_robot, 4 links, 3 joints
Links:
- added link caster_wheel, mass 0.2; visual sphere radius=0.05
Joints:
- added joint caster_wheel_joint: type continuous, parent base_link, child caster_wheel, origin xyz=0.15 0 -0.1 rpy=0 0 0, axis 0 0 1
- joint fixed_joint: origin xyz=0 0 0 -> xyz=0 0 0.15
- joint left_wheel_joint: origin xyz=-0.3 0.2 0 -> xyz=-0.175 0.255 -0.05 rpy=-1.5708 0 0
- joint right_wheel_joint: origin xyz=-0.3 -0.2 0 -> xyz=-.175 -0.255 -0.05 rpy=-1.5708 0 0
