Commit message: Completed visual for robot arm

File: src/my_robot_description/urdf/arm.xacro (robot description, xacro)
@@ -2,18 +2,18 @@
 <robot xmlns:xacro="http://www.ros.org/wiki/xacro">
     <!--add variables-->
-    <!--base footprint-->
-    <link name="base_footprint"/>
-    <joint name="base_joint" type="fixed">
-        <parent link="base_footprint"/>
-        <child link="arm_base_link"/>
-        <origin xyz="0 0 0" rpy="0 0 0"/> <!--fill in xyz-->
-    </joint>
+    <xacro:property name="arm_base_length" value="0.1"/>
+    <xacro:property name="arm_base_width" value="0.1"/>
+    <xacro:property name="arm_base_height" value="0.02"/>
+    <xacro:property name="forearm_radius" value="0.02"/>
+    <xacro:property name="forearm_length" value="0.3"/>
+    <xacro:property name="hand_radius" value="0.02" />
+    <xacro:property name="hand_length" value="0.3" />
     <!--base link add collision and inertia-->
     <link name="arm_base_link">
         <visual>
             <geometry>
-                <box size="0 0 0"/> <!--todo: add dimensions-->
+                <box size="${arm_base_length} ${arm_base_width} ${arm_base_height}"/>
             </geometry>
-            <origin xyz="0 0 0" rpy="0 0 0"/> <!--todo: xyz-->
+            <origin xyz="0 0 ${arm_base_height / 2.0}" rpy="0 0 0"/>
             <material name="orange"/>
         </visual>
@@ -23,8 +23,8 @@
         <visual>
             <geometry>
-                <cylinder radius="0" length="0"/><!--todo: add dimensions-->
-                <origin xyz="0 0 0" rpy="0 0 0"/> <!--add xyz-->
-                <material name="yellow"/>
+                <cylinder radius="${forearm_radius}" length="${forearm_length}"/>
             </geometry>
+            <origin xyz="0 0 ${forearm_length/2.0}" rpy="0 0 0"/>
+            <material name="yellow"/>
         </visual>
     </link>
@@ -33,18 +33,17 @@
         <visual>
             <geometry>
-                <cylinder radius="0" length="0"/> <!--todo: add dimensions-->
-                <origin xyz="0 0 0" rpy="0 0 0"/> <!--add xyz-->
-                <material name="orange"/>
+                <cylinder radius="${hand_radius}" length="${hand_length}"/>
             </geometry>
+            <origin xyz="0 0 ${hand_length/2.0}" rpy="0 0 0"/>
+            <material name="orange"/>
         </visual>
     </link>
     <!--forearm joint-->
     <joint name="forearm_joint" type="revolute">
-        <parent link="base_link"/>
+        <parent link="arm_base_link"/>
         <child link="forearm_link"/>
-        <origin xyz="0 0 0"/>
-        <axis xyz="0 0 0"/>
-        <limit lower="" upper="" effort="" velocity=""/> <!-- fill in from here up-->
-        <dynamics friction="0.05" damping="0.1"/>
+        <origin xyz="0 0 ${arm_base_height}" rpy="0 0 0"/>
+        <axis xyz="0 1 0"/>
+        <limit lower="0" upper="${pi/2}" effort="100" velocity="100"/>
     </joint>
     <!--hand joint-->
@@ -52,8 +51,7 @@
         <parent link="forearm_link"/>
         <child link="hand_link"/>
-        <origin xyz="0 0 0"/>
-        <axis xyz="0 0 0"/>
-        <limit lower="" upper="" effort="" velocity=""/> <!-- fill in from here up-->
-        <dynamics friction="0.05" damping="0.1"/>
+        <origin xyz="0 0 ${forearm_length}" rpy="0 0 0"/>
+        <axis xyz="0 1 0"/>
+        <limit lower="0" upper="${pi/2}" effort="100" velocity="100"/>
     </joint>
 </robot>

File: src/my_robot_description/urdf/standalone_arm.urdf.xacro (robot description, xacro)
@@ -1,4 +1,4 @@
 <?xml version="1.0"?>
-<robot name="my_robot" xmlns:xacro="http://www.ros.org/wiki/xacro">
+<robot name="my_robot_arm" xmlns:xacro="http://www.ros.org/wiki/xacro">
     <xacro:include filename="common_properties.xacro"/>
     <xacro:include filename="arm.xacro"/>

Commit message: added joint state publisher controller for the arm

File: src/my_robot_description/urdf/arm.xacro (robot description, xacro)
@@ -9,5 +9,5 @@
     <xacro:property name="hand_radius" value="0.02" />
     <xacro:property name="hand_length" value="0.3" />
-    <!--base link add collision and inertia-->
+    <!--base link add inertia-->
     <link name="arm_base_link">
         <visual>
@@ -18,6 +18,14 @@
             <material name="orange"/>
         </visual>
+        <collision>
+            <geometry>
+                <box size="${arm_base_length} ${arm_base_width} ${arm_base_height}"/>
+            </geometry>
+            <origin xyz="0 0 ${arm_base_height / 2.0}" rpy="0 0 0"/>
+        </collision>
+        <xacro:box_inertia m="0.5" l="${2*arm_base_length}" w="${2*arm_base_width}" h="${2*arm_base_height}"
+                            xyz="0 0 ${arm_base_height / 2.0}" rpy="0 0 0"/>
     </link>
-    <!--forearm link add collision and inertia-->
+    <!--forearm link add inertia-->
     <link name="forearm_link">
         <visual>
@@ -28,6 +36,14 @@
             <material name="yellow"/>
         </visual>
+        <collision>
+            <geometry>
+                <cylinder radius="${forearm_radius}" length="${forearm_length}"/>
+            </geometry>
+            <origin xyz="0 0 ${forearm_length/2.0}" rpy="0 0 0"/>
+        </collision>
+        <xacro:wheel_inertia m="0.3" r="${2*forearm_radius}" h="${2*forearm_length}"
+                                xyz="0 0 ${forearm_length/2.0}" rpy="0 0 0"/>
     </link>
-    <!--hand link-->
+    <!--hand link add inertia-->
     <link name="hand_link">
         <visual>
@@ -38,4 +54,12 @@
             <material name="orange"/>
         </visual>
+        <collision>
+            <geometry>
+                <cylinder radius="${hand_radius}" length="${hand_length}"/>
+            </geometry>
+            <origin xyz="0 0 ${hand_length/2.0}" rpy="0 0 0"/>
+        </collision>
+        <xacro:wheel_inertia m="0.3" r="${2*hand_radius}" h="${2*hand_length}"
+                                xyz="0 0 ${hand_length/2.0}" rpy="0 0 0"/>
     </link>
     <!--forearm joint-->
@@ -46,4 +70,5 @@
         <axis xyz="0 1 0"/>
         <limit lower="0" upper="${pi/2}" effort="100" velocity="100"/>
+        <dynamics friction="0.05" damping="0.1"/>
     </joint>
     <!--hand joint-->
@@ -54,4 +79,5 @@
         <axis xyz="0 1 0"/>
         <limit lower="0" upper="${pi/2}" effort="100" velocity="100"/>
+        <dynamics friction="0.05" damping="0.1"/>
     </joint>
 </robot>

File: src/my_robot_description/urdf/standalone_arm.urdf.xacro (robot description, xacro)
@@ -3,3 +3,4 @@
     <xacro:include filename="common_properties.xacro"/>
     <xacro:include filename="arm.xacro"/>
+    <xacro:include filename="arm_gazebo.xacro"/>
 </robot>
