Commit message: create variables with xacro properties

File: src/my_robot_description/urdf/my_robot.urdf.xacro (robot description, xacro)
@@ -1,4 +1,9 @@
 <?xml version="1.0"?>
-<robot name="my_robot">
+<robot name="my_robot" xmlns:xacro="http://www.ros.org/wiki/xacro">
+    <xacro:property name="base_length" value="0.6"/>
+    <xacro:property name="base_width" value="0.4"/>
+    <xacro:property name="base_height" value="0.2"/>
+    <xacro:property name="wheel_radius" value="0.1"/>
+    <xacro:property name="wheel_length" value="0.05"/>
     <!--define colors -->
     <material name="grey">
@@ -22,5 +27,5 @@
         <visual>
             <geometry>
-                <box size="0.6 0.4 0.2"/>
+                <box size="${base_length} ${base_width} ${base_height}"/>
             </geometry>
             <origin xyz="0 0 0.1" rpy="0 0 0"/>
@@ -47,5 +52,5 @@
         <visual>
             <geometry>
-                <cylinder radius="0.1" length="0.05"/>
+                <cylinder radius="${wheel_radius}" length="${wheel_length}"/>
             </geometry>
             <origin xyz="0 0 0" rpy="1.57 0 0"/>
@@ -56,5 +61,5 @@
         <parent link="base_link" />
         <child link="left_wheel" />
-        <origin xyz="-0.15 0.225 0" rpy="0 0 0"/>
+        <origin xyz="${-base_length/4.0} 0.225 0" rpy="0 0 0"/>
         <axis xyz="0 1 0" />
     </joint>
@@ -63,5 +68,5 @@
         <visual>
             <geometry>
-                <cylinder radius="0.1" length="0.05"/>
+                <cylinder radius="${wheel_radius}" length="${wheel_length}"/>
             </geometry>
             <origin xyz="0 0 0" rpy="1.57 0 0"/>
@@ -72,5 +77,5 @@
         <parent link="base_link" />
         <child link="right_wheel" />
-        <origin xyz="-0.15 -0.225 0" rpy="0 0 0"/>
+        <origin xyz="${-base_length/4.0} -0.225 0" rpy="0 0 0"/>
         <axis xyz="0 1 0" />
     </joint>
@@ -88,5 +93,5 @@
         <parent link="base_link" />
         <child link="caster_wheel" />
-        <origin xyz="0.2 0 -0.05" rpy="0 0 0"/>
+        <origin xyz="${base_length/3.0} 0 -0.05" rpy="0 0 0"/>
         <axis xyz="0 1 0" />
     </joint>

Commit message: created wheel functions with xacro macros

File: src/my_robot_description/urdf/my_robot.urdf.xacro (robot description, xacro)
@@ -19,7 +19,7 @@
     <link name="base_footprint"/>
     <joint name="base_joint" type="fixed">
-        <parent link="base_link"/>
-        <child link="base_footprint"/>
-        <origin xyz="0 0.1 0" rpy="0 0 0"/>
+        <parent link="base_footprint"/>
+        <child link="base_link"/>
+        <origin xyz="0 0 0.1" rpy="0 0 0"/>
     </joint>
     <!--base link-->
@@ -48,14 +48,19 @@
         <origin xyz="0 0 0.225" rpy="0 0 0"/>
     </joint>
+    <!--right wheel xacro macro-->
+    <xacro:macro name="wheel" params="prefix">
+        <link name="${prefix}_wheel">
+            <visual>
+                <geometry>
+                    <cylinder radius="${wheel_radius}" length="${wheel_length}"/>
+                </geometry>
+                <origin xyz="0 0 0" rpy="1.57 0 0"/>
+                <material name="grey"/>
+            </visual>
+        </link>
+    </xacro:macro>
+    <xacro:wheel prefix="right" />
+    <xacro:wheel prefix="left" />
     <!--left wheel-->
-    <link name="left_wheel">
-        <visual>
-            <geometry>
-                <cylinder radius="${wheel_radius}" length="${wheel_length}"/>
-            </geometry>
-            <origin xyz="0 0 0" rpy="1.57 0 0"/>
-            <material name="grey"/>
-        </visual>
-    </link>
     <joint name="left_wheel_link" type="continuous">
         <parent link="base_link" />
@@ -65,13 +70,4 @@
     </joint>
     <!--right wheel-->
-    <link name="right_wheel">
-        <visual>
-            <geometry>
-                <cylinder radius="${wheel_radius}" length="${wheel_length}"/>
-            </geometry>
-            <origin xyz="0 0 0" rpy="1.57 0 0"/>
-            <material name="grey"/>
-        </visual>
-    </link>
     <joint name="right_wheel_link" type="continuous">
         <parent link="base_link" />

Commit message: Separated the urdf into multiple xacro files

File: src/my_robot_description/urdf/my_robot.urdf.xacro (robot description, xacro)
@@ -1,94 +1,5 @@
 <?xml version="1.0"?>
 <robot name="my_robot" xmlns:xacro="http://www.ros.org/wiki/xacro">
-    <xacro:property name="base_length" value="0.6"/>
-    <xacro:property name="base_width" value="0.4"/>
-    <xacro:property name="base_height" value="0.2"/>
-    <xacro:property name="wheel_radius" value="0.1"/>
-    <xacro:property name="wheel_length" value="0.05"/>
-    <!--define colors -->
-    <material name="grey">
-        <color rgba="0.7 0.7 0.7 1"/>
-    </material>
-    <material name="green">
-        <color rgba="0 0.6 0.0 1"/>
-    </material>
-    <material name="white">
-        <color rgba="1 1 1 1" />
-    </material>
-    <!--base footprint-->
-    <link name="base_footprint"/>
-    <joint name="base_joint" type="fixed">
-        <parent link="base_footprint"/>
-        <child link="base_link"/>
-        <origin xyz="0 0 0.1" rpy="0 0 0"/>
-    </joint>
-    <!--base link-->
-    <link name="base_link">
-        <visual>
-            <geometry>
-                <box size="${base_length} ${base_width} ${base_height}"/>
-            </geometry>
-            <origin xyz="0 0 0.1" rpy="0 0 0"/>
-            <material name="green"/>
-        </visual>
-    </link>
-    <!-- lidar -->
-    <link name="lidar">
-        <visual>
-            <geometry>
-                <cylinder radius="0.1" length="0.05"/>
-            </geometry>
-            <origin xyz="0 0 0" rpy="0 0 0" />
-            <material name="white"/>
-        </visual>
-    </link>
-    <joint name="base_lidar_joint" type="fixed">
-        <parent link="base_link" />
-        <child link="lidar" />
-        <origin xyz="0 0 0.225" rpy="0 0 0"/>
-    </joint>
-    <!--right wheel xacro macro-->
-    <xacro:macro name="wheel" params="prefix">
-        <link name="${prefix}_wheel">
-            <visual>
-                <geometry>
-                    <cylinder radius="${wheel_radius}" length="${wheel_length}"/>
-                </geometry>
-                <origin xyz="0 0 0" rpy="1.57 0 0"/>
-                <material name="grey"/>
-            </visual>
-        </link>
-    </xacro:macro>
-    <xacro:wheel prefix="right" />
-    <xacro:wheel prefix="left" />
-    <!--left wheel-->
-    <joint name="left_wheel_link" type="continuous">
-        <parent link="base_link" />
-        <child link="left_wheel" />
-        <origin xyz="${-base_length/4.0} 0.225 0" rpy="0 0 0"/>
-        <axis xyz="0 1 0" />
-    </joint>
-    <!--right wheel-->
-    <joint name="right_wheel_link" type="continuous">
-        <parent link="base_link" />
-        <child link="right_wheel" />
-        <origin xyz="${-base_length/4.0} -0.225 0" rpy="0 0 0"/>
-        <axis xyz="0 1 0" />
-    </joint>
-    <!--caster wheel-->
-    <link name="caster_wheel">
-        <visual>
-            <geometry>
-                <sphere radius="0.05"/>
-            </geometry>
-            <origin xyz="0 0 0" rpy="0 0 0"/>
-            <material name="grey"/>
-        </visual>
-    </link>
-    <joint name="caster_wheel_link" type="fixed">
-        <parent link="base_link" />
-        <child link="caster_wheel" />
-        <origin xyz="${base_length/3.0} 0 -0.05" rpy="0 0 0"/>
-        <axis xyz="0 1 0" />
-    </joint>
+    <xacro:include filename="common_properties.xacro"/>
+    <xacro:include filename="mobile_base.xacro"/>
 </robot>

Commit message: Completed three wheeled robot with robot arm on top

File: src/my_robot_description/urdf/my_robot.urdf.xacro (robot description, xacro)
@@ -4,4 +4,11 @@
     <xacro:include filename="mobile_base.xacro"/>
     <xacro:include filename="mobile_base_gazebo.xacro"/>
-    <xacro:include filename="camera.xacro"/>
+    <xacro:include filename="arm.xacro"/>
+    <xacro:include filename="arm_gazebo.xacro"/>
+    <joint name="mobile_base_arm_joint" type="fixed">
+        <parent link="base_link"/>
+        <child link="arm_base_link"/>
+        <origin xyz="${base_length/4} 0 ${base_height}" rpy="0 0 0"/>
+    </joint>
+    <!--<xacro:include filename="camera.xacro"/>-->
 </robot>
