Commit message: Added camera to the robot and a camera plugin

File: src/my_robot_description/urdf/camera.xacro (robot description, xacro)
@@ -24,3 +24,14 @@
         <origin xyz="${(base_length + camera_length) /2.0} 0 ${base_height/2}" rpy="0 0 0"/>
     </joint>
+    <gazebo reference="camera_link">
+        <material>Gazebo/Red</material>
+        <sensor name="camera_sensor" type="camera">
+            <pose>0 0 0 0 0 0</pose>
+            <visualize>true</visualize>
+            <update_rate>10.0</update_rate>
+            <plugin name="camera_controller" filename="libgazebo_ros_camera.so">
+                <frame_name>camera_link</frame_name>
+            </plugin>
+        </sensor>
+    </gazebo>
 </robot>

Commit message: velocity controller to move robot in a striaght line

File: src/my_robot_description/urdf/camera.xacro (robot description, xacro)
@@ -13,5 +13,5 @@
         <collision>
             <geometry>
-                <box size="${camera_length} ${camera_width} {camera_height}"/>
+                <box size="${camera_length} ${camera_width} ${camera_height}"/>
             </geometry>
         </collision>

File: src/my_robot_description/urdf/common_properties.xacro (robot description, xacro)
@@ -16,4 +16,7 @@
     <material name="yellow">
         <color rgba="1 1 0 1"/>
+    </material>
+    <material name="blue">
+        <color rgba="0 0 1 1"/>
     </material>
     <xacro:macro name="box_inertia" params="m l w h xyz rpy">

File: src/my_robot_description/urdf/my_robot.urdf.xacro (robot description, xacro)
@@ -4,5 +4,6 @@
     <xacro:include filename="mobile_base.xacro"/>
     <xacro:include filename="mobile_base_gazebo.xacro"/>
-    <xacro:include filename="arm.xacro"/>
+    <xacro:include filename="camera.xacro"/>
+    <!--<xacro:include filename="arm.xacro"/>
     <xacro:include filename="arm_gazebo.xacro"/>
     <joint name="mobile_base_arm_joint" type="fixed">
@@ -10,5 +11,4 @@
         <child link="arm_base_link"/>
         <origin xyz="${base_length/4} 0 ${base_height}" rpy="0 0 0"/>
-    </joint>
-    <!--<xacro:include filename="camera.xacro"/>-->
+    </joint>-->
 </robot>
