Commit message: fixed stop and go behavior of robot when moving forward

File: src/my_robot_description/urdf/mobile_base_gazebo.xacro (robot description, xacro)
@@ -20,6 +20,6 @@
             <update_rate>50</update_rate>
             <!-- wheels -->
-            <left_joint>left_wheel_link</left_joint>
-            <right_joint>right_wheel_link</right_joint>
+            <left_joint>base_left_wheel_joint</left_joint>
+            <right_joint>base_right_wheel_joint</right_joint>
             <!-- kinematics -->
             <wheel_separation>0.45</wheel_separation>

File: src/my_robot_description/urdf/my_robot.urdf.xacro (robot description, xacro)
@@ -4,3 +4,4 @@
     <xacro:include filename="mobile_base.xacro"/>
     <xacro:include filename="mobile_base_gazebo.xacro"/>
+    <xacro:include filename="camera.xacro"/>
 </robot>

File: src/my_robot_description/urdf/temp_mobile_base.xacro (robot description, xacro)
@@ -11,5 +11,5 @@
         <parent link="base_footprint"/>
         <child link="base_link"/>
-        <origin xyz="0 0 ${wheel_radius}" rpy="0 0 0"/>
+        <origin xyz="0 0 0.1" rpy="0 0 0"/>
     </joint>
     <!--base link-->
@@ -19,6 +19,6 @@
                 <box size="${base_length} ${base_width} ${base_height}"/>
             </geometry>
-            <origin xyz="0 0 ${base_height / 2.0}" rpy="0 0 0"/>
-            <material name="blue"/>
+            <origin xyz="0 0 0.1" rpy="0 0 0"/>
+            <material name="green"/>
         </visual>
         <collision>
@@ -26,50 +26,50 @@
                 <box size="${base_length} ${base_width} ${base_height}"/>
             </geometry>
-            <origin xyz="0 0 ${base_height / 2.0}" rpy="0 0 0"/>
+            <origin xyz="0 0 0.1" rpy="0 0 0"/>
         </collision>
         <xacro:box_inertia m="5.0" l="${2*base_length}" w="${2*base_width}" h="${2*base_height}"
-                            xyz="0 0 ${base_height / 2.0}" rpy="0 0 0"/>
+                            xyz="0 0 0.1" rpy="0 0 0"/>
     </link>
     <!--wheel xacro macro-->
-    <xacro:macro name="wheel_link" params="prefix">
-        <link name="${prefix}_wheel_link">
+    <xacro:macro name="wheel" params="prefix">
+        <link name="${prefix}_wheel">
             <visual>
                 <geometry>
                     <cylinder radius="${wheel_radius}" length="${wheel_length}"/>
                 </geometry>
-                <origin xyz="0 0 0" rpy="${pi / 2.0} 0 0"/>
+                <origin xyz="0 0 0" rpy="1.57 0 0"/>
                 <material name="grey"/>
             </visual>
             <collision>
                 <geometry>
-                    <sphere radius="${wheel_radius}" length="${wheel_length}"/>
+                    <sphere radius="0.1"/>
                 </geometry>
-                <origin xyz="0 0 0" rpy="${pi / 2.0} 0 0"/>
+                <origin xyz="0 0 0" rpy="0 0 0"/>
             </collision>
             <xacro:wheel_inertia m="1.0" r="${2*wheel_radius}" h="${2*wheel_length}"
-                                xyz="0 0 0" rpy="${pi / 2.0} 0 0"/>
+                                xyz="0 0 0" rpy="1.57 0 0"/>
         </link>
     </xacro:macro>
-    <xacro:wheel_link prefix="right" />
-    <xacro:wheel_link prefix="left" />
+    <xacro:wheel prefix="right" />
+    <xacro:wheel prefix="left" />
     <!--left wheel-->
     <joint name="base_left_wheel_joint" type="continuous">
         <parent link="base_link" />
-        <child link="left_wheel_link" />
-        <origin xyz="${-base_length / 4.0} ${(base_width + wheel_length) / 2.0} 0" rpy="0 0 0"/>
+        <child link="left_wheel" />
+        <origin xyz="${-base_length/4.0} 0.225 0" rpy="0 0 0"/>
         <axis xyz="0 1 0" />
     </joint>
     <!--right wheel-->
-    <joint name="base_right_wheel_joint" type="continuous">
+    <joint name="base_right_wheel_join" type="continuous">
         <parent link="base_link" />
-        <child link="right_wheel_link" />
-        <origin xyz="${-base_length / 4.0} ${-(base_width + wheel_length) / 2.0} 0" rpy="0 0 0"/>
+        <child link="right_wheel" />
+        <origin xyz="${-base_length/4.0} -0.225 0" rpy="0 0 0"/>
         <axis xyz="0 1 0" />
     </joint>
     <!--caster wheel-->
-    <link name="caster_wheel_link">
+    <link name="caster_wheel">
         <visual>
             <geometry>
-                <sphere radius="${wheel_radius / 2.0}"/>
+                <sphere radius="0.05"/>
             </geometry>
             <origin xyz="0 0 0" rpy="0 0 0"/>
@@ -78,5 +78,5 @@
         <collision>
             <geometry>
-                <sphere radius="${wheel_radius / 2.0}"/>
+                <sphere radius="0.05"/>
             </geometry>
             <origin xyz="0 0 0" rpy="0 0 0"/>
@@ -87,5 +87,5 @@
     <joint name="caster_wheel_link" type="fixed">
         <parent link="base_link" />
-        <child link="caster_wheel_link" />
+        <child link="caster_wheel" />
         <origin xyz="${base_length/3.0} 0 ${-wheel_radius / 2.0}" rpy="0 0 0"/>
     </joint>

Commit message: added a sim_time parameter to launch file to synchronize time between nodes in Gazebo

File: src/my_robot_description/urdf/mobile_base_gazebo.xacro (robot description, xacro)
@@ -15,25 +15,28 @@
         <mu2 value="0.1" />
     </gazebo>
-    <gazebo>
-        <plugin name="gazebo_ros2_control" filename="libgazebo_ros2_control.so"/>
-    </gazebo>
+   <!-- <gazebo>
+        <plugin name="simple_controller" filename="libgazebo_ros_basic_controller.so">
+            <joint name="base_right_wheel_joint"/>
+            <joint name="base_left_wheel_joint"/>
+        </plugin>
+    </gazebo>-->
     <gazebo>
         <plugin name="diff_drive_controller" filename="libgazebo_ros_diff_drive.so">
-            <!-- Update rate in Hz -->
+            <!--Update rate in Hz -->
             <update_rate>50</update_rate>
-            <!-- wheels -->
+             <!--wheels -->
             <left_joint>base_left_wheel_joint</left_joint>
             <right_joint>base_right_wheel_joint</right_joint>
-            <!-- kinematics -->
-            <wheel_separation>0.45</wheel_separation>
-            <wheel_diameter>0.2</wheel_diameter>
-            <!-- output -->
-            <publish_odom>true</publish_odom>
-            <publish_odom_tf>true</publish_odom_tf>
-            <publish_wheel_tf>true</publish_wheel_tf>
-            <odometry_topic>odom</odometry_topic>
-            <odometry_frame>odom</odometry_frame>
-            <robot_base_frame>base_footprint</robot_base_frame>
-        </plugin>
-    </gazebo>
+             <!--kinematics-->
+             <wheel_separation>0.45</wheel_separation>
+             <wheel_diameter>0.2</wheel_diameter>
+             <!--output -->
+             <publish_odom>true</publish_odom>
+             <publish_odom_tf>true</publish_odom_tf>
+             <publish_wheel_tf>true</publish_wheel_tf>
+             <odometry_topic>odom</odometry_topic>
+             <odometry_frame>odom</odometry_frame>
+             <robot_base_frame>base_footprint</robot_base_frame>
+         </plugin>
+     </gazebo>
 </robot>
