Commit message: added inertia macros to the urdf

File: src/my_robot_description/urdf/common_properties.xacro (robot description, xacro)
@@ -11,3 +11,30 @@
         <color rgba="1 1 1 1" />
     </material>
+    <xacro:macro name="box_inertia" params="m l w h xyz rpy">
+        <inertial>
+            <origin xyz="${xyz}" rpy="${rpy}"/>
+            <mass value="${m}"/>
+            <inertia ixx = "${(m/12) * (h*h + l*l)}" ixy="0" ixz="0"
+                    iyy="${(m/12) * (w*w = l*l)}" iyz="0"
+                    izz="{(m/12) * (w*w + h*h)}"/>
+        </inertial>
+    </xacro:macro>
+    <xacro:macro name="wheel_inertia" params="m r h xyz rpy">
+        <inertial>
+            <origin xyz="${xyz}" rpy="${rpy}"/>
+            <mass value="${m}"/>
+            <inertia ixx="${(m/12) * (3*r*r + h*h)}"  ixy="0" ixz="0"
+                    iyy="${(m/12) * (3*r*r + h*h)}" iyz="0"
+                    izz="${(m/2) * (r * r)}"/>
+        </inertial>
+    </xacro:macro>
+    <xacro:macro name="caster_wheel_inertia" params="m r xyz rpy">
+        <inertial>
+            <origin xyz="${xyz}" rpy="${rpy}"/>
+            <mass value="${m}"/>
+            <inertia ixx="${2/5 * (m * r * r)}" ixy="0" ixz="0"
+                    iyy="${2/5 * (m * r * r)}" iyz="0"
+                    izz="${2/5 * (m * r * r)}"/>
+        </inertial>
+    </xacro:macro>
 </robot>

File: src/my_robot_description/urdf/mobile_base.xacro (robot description, xacro)
@@ -22,4 +22,6 @@
             <material name="green"/>
         </visual>
+        <xacro:box_inertia m="5.0" l="${base_length}" w="{base_width}" h="{base_height}"
+                            xyz="0 0 ${base_height}/2" rpy="0 0 0"/>
     </link>
     <!-- lidar -->
@@ -32,4 +34,6 @@
             <material name="white"/>
         </visual>
+        <xacro:wheel_inertia m="1.0" r="${wheel_radius}" h="${wheel_length}"
+                            xyz="0 0 0" rpy="0 0 0"/>
     </link>
     <joint name="base_lidar_joint" type="fixed">
@@ -38,5 +42,5 @@
         <origin xyz="0 0 0.225" rpy="0 0 0"/>
     </joint>
-    <!--right wheel xacro macro-->
+    <!--wheel xacro macro-->
     <xacro:macro name="wheel" params="prefix">
         <link name="${prefix}_wheel">
@@ -48,4 +52,6 @@
                 <material name="grey"/>
             </visual>
+            <xacro:wheel_inertia m="1.0" r="${wheel_radius}" h="${wheel_length}"
+                                xyz="0 0 0" rpy="1.57 0 0"/>
         </link>
     </xacro:macro>
@@ -75,4 +81,6 @@
             <material name="grey"/>
         </visual>
+        <xacro:caster_wheel_inertia m="0.5" r="${wheel_radius/2}"
+                                    xyz="0 0 0" rpy="0 0 0"/>
     </link>
     <joint name="caster_wheel_link" type="fixed">

Commit message: Added collision tags to urdf

File: src/my_robot_description/urdf/common_properties.xacro (robot description, xacro)
@@ -16,6 +16,6 @@
             <mass value="${m}"/>
             <inertia ixx = "${(m/12) * (h*h + l*l)}" ixy="0" ixz="0"
-                    iyy="${(m/12) * (w*w = l*l)}" iyz="0"
-                    izz="{(m/12) * (w*w + h*h)}"/>
+                    iyy="${(m/12) * (w*w + l*l)}" iyz="0"
+                    izz="${(m/12) * (w*w + h*h)}"/>
         </inertial>
     </xacro:macro>
@@ -24,7 +24,7 @@
             <origin xyz="${xyz}" rpy="${rpy}"/>
             <mass value="${m}"/>
-            <inertia ixx="${(m/12) * (3*r*r + h*h)}"  ixy="0" ixz="0"
-                    iyy="${(m/12) * (3*r*r + h*h)}" iyz="0"
-                    izz="${(m/2) * (r * r)}"/>
+            <inertia ixx="${(m/12) * (3.0*r*r + h*h)}"  ixy="0" ixz="0"
+                    iyy="${(m/12) * (3.0*r*r + h*h)}" iyz="0"
+                    izz="${(m/2) * (r*r)}"/>
         </inertial>
     </xacro:macro>
@@ -33,7 +33,7 @@
             <origin xyz="${xyz}" rpy="${rpy}"/>
             <mass value="${m}"/>
-            <inertia ixx="${2/5 * (m * r * r)}" ixy="0" ixz="0"
-                    iyy="${2/5 * (m * r * r)}" iyz="0"
-                    izz="${2/5 * (m * r * r)}"/>
+            <inertia ixx="${(2/5) * m * r * r}" ixy="0" ixz="0"
+                    iyy="${(2/5) * m * r * r}" iyz="0"
+                    izz="${(2/5) * m * r * r}"/>
         </inertial>
     </xacro:macro>

File: src/my_robot_description/urdf/mobile_base.xacro (robot description, xacro)
@@ -22,8 +22,14 @@
             <material name="green"/>
         </visual>
-        <xacro:box_inertia m="5.0" l="${base_length}" w="{base_width}" h="{base_height}"
-                            xyz="0 0 ${base_height}/2" rpy="0 0 0"/>
+        <collision>
+            <geometry>
+                <box size="${base_length} ${base_width} ${base_height}"/>
+            </geometry>
+            <origin xyz="0 0 0.1" rpy="0 0 0"/>
+        </collision>
+        <xacro:box_inertia m="5.0" l="${base_length}" w="${base_width}" h="${base_height}"
+                            xyz="0 0 0.1" rpy="0 0 0"/>
     </link>
-    <!-- lidar -->
+    <!-- lidar
     <link name="lidar">
         <visual>
@@ -41,5 +47,5 @@
         <child link="lidar" />
         <origin xyz="0 0 0.225" rpy="0 0 0"/>
-    </joint>
+    </joint>-->
     <!--wheel xacro macro-->
     <xacro:macro name="wheel" params="prefix">
@@ -52,4 +58,10 @@
                 <material name="grey"/>
             </visual>
+            <collision>
+                <geometry>
+                    <sphere radius="0.1"/>
+                </geometry>
+                <origin xyz="0 0 0" rpy="0 0 0"/>
+            </collision>
             <xacro:wheel_inertia m="1.0" r="${wheel_radius}" h="${wheel_length}"
                                 xyz="0 0 0" rpy="1.57 0 0"/>
@@ -81,5 +93,11 @@
             <material name="grey"/>
         </visual>
-        <xacro:caster_wheel_inertia m="0.5" r="${wheel_radius/2}"
+        <collision>
+            <geometry>
+                <sphere radius="0.05"/>
+            </geometry>
+            <origin xyz="0 0 0" rpy="0 0 0"/>
+        </collision>
+        <xacro:caster_wheel_inertia m="0.5" r="${wheel_radius/2.0}"
                                     xyz="0 0 0" rpy="0 0 0"/>
     </link>
@@ -88,5 +106,4 @@
         <child link="caster_wheel" />
         <origin xyz="${base_length/3.0} 0 -0.05" rpy="0 0 0"/>
-        <axis xyz="0 1 0" />
     </joint>
 </robot>

Commit message: added links and joints to arm urdf and removed temp files

File: src/my_robot_description/urdf/common_properties.xacro (robot description, xacro)
@@ -10,4 +10,10 @@
     <material name="white">
         <color rgba="1 1 1 1" />
+    </material>
+    <material name="orange">
+        <color rgba="1 0.647 0 1"/>
+    </material>
+    <material name="yellow">
+        <color rgba="1 1 0 1"/>
     </material>
     <xacro:macro name="box_inertia" params="m l w h xyz rpy">

Commit message: fixed errors with lidar and imu

File: src/my_robot_description/urdf/common_properties.xacro (robot description, xacro)
@@ -19,4 +19,7 @@
     <material name="blue">
         <color rgba="0 0 1 1"/>
+    </material>
+    <material name="black">
+        <color rgba="0 0 0 0"/>
     </material>
     <xacro:macro name="box_inertia" params="m l w h xyz rpy">

File: src/my_robot_description/urdf/mobile_base.xacro (robot description, xacro)
@@ -121,3 +121,24 @@
         <origin xyz="0 0 0.225"/>
     </joint>
+    <!--IMU-->
+    <link name="imu_link">
+        <visual>
+            <geometry>
+                <box size="0.05 0.05 0.02"/>
+            </geometry>
+            <material name="grey"/>
+        </visual>
+        <sensor name="imu_sensor" type="imu">
+            <origin xyz="0 0 0.1"/>
+            <imu>
+                <always_on>true</always_on>
+                <update_rate>50</update_rate>
+            </imu>
+        </sensor>
+    </link>
+    <joint name="imu_joint" type="fixed">
+        <parent link="base_link"/>
+        <child link="imu_link"/>
+        <origin xyz="0 0 0.015"/>
+    </joint>
 </robot>

File: src/my_robot_description/urdf/mobile_base_gazebo.xacro (robot description, xacro)
@@ -15,10 +15,34 @@
         <mu2 value="0.1" />
     </gazebo>
-   <!-- <gazebo>
-        <plugin name="simple_controller" filename="libgazebo_ros_basic_controller.so">
-            <joint name="base_right_wheel_joint"/>
-            <joint name="base_left_wheel_joint"/>
-        </plugin>
-    </gazebo>-->
+    <gazebo reference="lidar_link">
+        <sensor type="ray" name="lidar_sensor">
+            <update_rate>10</update_rate>
+            <ray>
+                <scan>
+                    <horizontal>
+                        <samples>360</samples>
+                        <resolution>1</resolution>
+                        <min_angle>-1.57</min_angle>
+                        <max_angle>1.57</max_angle>
+                    </horizontal>
+                </scan>
+                <range>
+                    <min>0.1</min>
+                    <max>10.0</max>
+                </range>
+            </ray>
+            <plugin name="gazebo_ros_laser" filename="libgazebo_ros_ray_sensor.so">
+                <ros>
+                    <namespace>/</namespace>
+                    <remapping>scan:=/scan</remapping>
+                </ros>
+            </plugin>
+        </sensor>
+    </gazebo>
+    <gazebo reference = "imu_sensor">
+        <sensor type="imu" name="imu_sensor">
+            <update_rate>50</update_rate>
+        </sensor>
+    </gazebo>
     <gazebo>
         <plugin name="diff_drive_controller" filename="libgazebo_ros_diff_drive.so">
